Commit message: collision updated (xacro)
Update crawer base

File: catkin_ws/src/arm_description/urdf/arm.urdf.xacro (robot description, xacro)
@@ -37,5 +37,5 @@
     <collision>
       <geometry>
-          <box size="0.05 0.08 0.1"/>
+          <box size="0.065 0.08 0.01"/>
       </geometry>
       <origin rpy="0 0 0" xyz="0 0.012 0.001"/>
@@ -86,7 +86,7 @@
     <collision>
       <geometry>
-           <box size="0.08 0.035 0.045"/>
-        </geometry>
-      <origin rpy="0 0 0" xyz="0 0 0"/>
+           <box size="0.055 0.035 0.045"/>
+        </geometry>
+      <origin rpy="0 0 0" xyz="0.012 0 0"/>
     </collision>
      <inertial>
@@ -146,7 +146,7 @@
    <collision>
       <geometry>
-          <box size="0.08 0.035 0.045"/>
-        </geometry>
-      <origin rpy="0 0 0" xyz="0 0 0"/>
+           <box size="0.055 0.035 0.045"/>
+        </geometry>
+      <origin rpy="0 0 0" xyz="0.012 0 0"/>
     </collision>
      <inertial>
@@ -205,7 +205,7 @@
     <collision>
       <geometry>
-          <box size="0.08 0.035 0.045"/>
-        </geometry>
-      <origin rpy="0 0 0" xyz="0 0 0"/>
+           <box size="0.055 0.035 0.045"/>
+        </geometry>
+      <origin rpy="0 0 0" xyz="0.012 0 0"/>
     </collision>
     <inertial>
@@ -264,7 +264,7 @@
     <collision>
       <geometry>
-          <box size="0.08 0.035 0.045"/>
-        </geometry>
-      <origin rpy="0 0 0" xyz="0 0 0"/>
+           <box size="0.055 0.035 0.045"/>
+        </geometry>
+      <origin rpy="0 0 0" xyz="0.012 0 0"/>
     </collision>
     <inertial>
